File: eeg_ble_pcb_v1.kicad_sch (KiCad schematic)
At the start: 37 parts, among them J1 USB_C_Receptacle_USB2.0_16P, Q1 FS8205, SW1 SW_Push, U1 STM32WB55RGVx, U2 DW01A, U2 TP4056-42-ESOP8, X1 NX2016SA-32MHZ-EXS00A-CS06654

Commit message: ADC, Buck, Boost, and charging unit added
Parts:
- added Bias, JP1, JP10, JP11, JP12, JP13, JP14, JP15, JP16, JP17, JP2, JP3, JP4, JP5, JP6, JP7, JP8: 0, Connector_PinHeader_2.54mm:PinHeader_1x02_P2.54mm_Vertical, symbol Libraryv2:SolderJumper_2_Open
- added C17: 100u, Capacitor_SMD:C_0805_2012Metric_Pad1.18x1.45mm_HandSolder, symbol Libraryv2:C_1
- added C17: 1n, Capacitor_SMD:C_0805_2012Metric_Pad1.18x1.45mm_HandSolder, symbol Libraryv2:C
- added C18 (x2), C19, C20, C21, C22 (x2), C26, C27, C28, C29, C30, C35: 1u, Capacitor_SMD:C_0805_2012Metric_Pad1.18x1.45mm_HandSolder, symbol Libraryv2:C_1
- added C23 (x2), C24, C34: 0.1u, Capacitor_SMD:C_0805_2012Metric_Pad1.18x1.45mm_HandSolder, symbol Libraryv2:C_1
- added C25: 10u, Capacitor_SMD:C_0805_2012Metric_Pad1.18x1.45mm_HandSolder, symbol Libraryv2:C_1
- added C31, C32, C33 (x2): 22u, Capacitor_SMD:C_0805_2012Metric_Pad1.18x1.45mm_HandSolder, symbol Libraryv2:C
- added C32: 10n, Capacitor_SMD:C_0805_2012Metric_Pad1.18x1.45mm_HandSolder, symbol Libraryv2:C
- added C36, C38, C39: 10u, Capacitor_SMD:C_0805_2012Metric_Pad1.18x1.45mm_HandSolder, symbol Libraryv2:C
- added C37: 0.1u, Capacitor_SMD:C_0805_2012Metric_Pad1.18x1.45mm_HandSolder, symbol Libraryv2:C
- added D5(5mm)1: LED, LED_SMD:LED_0805_2012Metric_Pad1.15x1.40mm_HandSolder, symbol Libraryv2:LED
- added L1: 1u, Inductor_SMD:L_0805_2012Metric_Pad1.15x1.40mm_HandSolder, symbol Libraryv2:L
- added L2: 2.2u, Inductor_SMD:L_0805_2012Metric_Pad1.15x1.40mm_HandSolder, symbol Libraryv2:L
- added R10, R11, R12, R13, R14, R15, R16, R17, R18, R19, R20, R21, R22, R23, R24, R29: 3.3k, Resistor_SMD:R_0805_2012Metric_Pad1.20x1.40mm_HandSolder, symbol Libraryv2:R
- added R25, R26, R27, R28, R30, R32: 100, Resistor_SMD:R_0805_2012Metric_Pad1.20x1.40mm_HandSolder, symbol Libraryv2:R
- added R30: 100k, Resistor_SMD:R_0805_2012Metric_Pad1.20x1.40mm_HandSolder, symbol Libraryv2:R
- added R31, R9: 1M, Resistor_SMD:R_0805_2012Metric_Pad1.20x1.40mm_HandSolder, symbol Libraryv2:R
- added R31: 402k, Resistor_SMD:R_0805_2012Metric_Pad1.20x1.40mm_HandSolder, symbol Libraryv2:R
- added SW2: SW_Push, Button_Switch_THT:SW_DIP_SPSTx01_Slide_6.7x4.1mm_W7.62mm_P2.54mm_LowProfile, symbol Libraryv2:SW_Push
- added U3: ADS1299-4PAGR, Library:QFP50P1200X1200X120-64N, symbol Libraryv2:ADS1299-4PAGR
- added U4: TPS61230DRC, Package_SON:Texas_S-PVSON-N10_ThermalVias, symbol Libraryv2:TPS61230DRC
- added U5: TPS63001, Package_SON:Texas_DRC0010J, symbol Libraryv2:TPS63001
Connections:
- net B+: now also SW2.1
- net GND renamed DGND
- net DGND: now also Bias.1 (A), C17.2, C18.2, C22.2, C22.2, C23.2, C23.2, C24.2, C25.2, C26.2, C31.2, C32.2, C33.2, C34.2, C35.2, C36.2, C37.2, C38.1, C38.2, C39.1, C39.2, JP1.1 (A), JP10.1 (A), JP11.1 (A), JP12.1 (A), JP13.1 (A), JP14.1 (A), JP15.1 (A), JP16.1 (A), JP17.1 (A), JP2.1 (A), JP3.1 (A), JP4.1 (A), JP5.1 (A), JP6.1 (A), JP7.1 (A), JP8.1 (A), R30.2, U3.20 (AVSS@1), U3.23 (AVSS@1), U3.25 (VREFN), U3.31 (RESV1), U3.32 (AVSS@1), U3.33 (DGND), U3.41 (DAISY_IN), U3.48 (DVDD), U3.49 (DGND), U3.50 (DVDD), U3.51 (DGND), U3.52 (CLKSEL), U3.53 (AVSS1), U3.57 (AVSS@1), U3.58 (AVSS@2), U4.11 (GND), U5.1 (VOUT), U5.10 (FB), U5.11 (PGND), U5.3 (PGND), U5.9 (GND)
- new net: JP17.2 (B), R29.1
- new net: JP16.2 (B), R16.1
- new net: C24.1, C25.1, U3.24 (VREFP)
- new net: JP6.2 (B), R22.1
- new net: L2.1, U5.2 (L2)
- new net: L2.2, U5.4 (L1)
- new net: JP12.2 (B), R12.1
- new net: C28.1, R12.2, U3.3 (IN7N)
- new net: C20.2, R22.2, U3.14 (IN2P)
- new net: JP11.2 (B), R11.1
- new net: C27.2, R11.2, U3.2 (IN8P)
- new net: C31.1, L1.1, R30.2, U4.10 (VIN), U4.9 (EN)
- new net: L1.2, U4.1 (SW), U4.2 (SW)
- new net: JP5.2 (B), R21.1
- new net: C20.1, R21.2, U3.13 (IN2N)
- new net: C18.1, R17.2, U3.9 (IN4N)
- new net: C18.2, R18.2, U3.10 (IN4P)
- new net: C32.2, C33.1
- new net: R31.1, U4.5 (PG)
- new net: R28.1, U3.34 (DIN)
- new net: C37.1, R32.2, U5.6 (EN), U5.7 (PS/SYNC), U5.8 (VINA)
- new net: C27.1, R10.2, U3.1 (IN8N)
- new net: C19.1, R19.2, U3.11 (IN3N)
- new net: C19.2, R20.2, U3.12 (IN3P)
- new net: C21.1, R23.2, U3.15 (IN1N)
- new net: C21.2, R24.2, U3.16 (IN1P)
- new net: C26.1, U3.26 (VCAP4)
- new net: C17.1, U3.28 (VCAP1)
- new net: C18.1, U3.30 (VCAP2)
- new net: R27.1, U3.38 (START)
- new net: R26.1, U3.39 (~{CS})
- new net: C28.2, R13.2, U3.4 (IN7P)
- new net: R25.1, U3.40 (SCLK)
- new net: C29.1, R14.2, U3.5 (IN6N)
- new net: C22.1, C23.1, U3.55 (VCAP3)
- new net: C29.2, R15.2, U3.6 (IN6P)
- new net: C17.2, R9.2, U3.61 (BIASINV)
- new net: Bias.2 (B), C17.1, R9.1, U3.62 (BIASIN), U3.63 (BIASOUT)
- new net: C30.1, R16.2, U3.7 (IN5N)
- new net: C30.2, R29.2, U3.8 (IN5P)
- new net: JP13.2 (B), R13.1
- new net: C32.1, C33.2
- new net: JP3.2 (B), R19.1
- new net: JP4.2 (B), R20.1
- new net: JP8.2 (B), R24.1
- new net: JP1.2 (B), R18.1
- new net: JP10.2 (B), R10.1
- new net: JP2.2 (B), R17.1
- new net: R30.1, R31.2, U4.7 (FB)
- new net: D5(5mm)1.1 (K), R30.1
- new net: D5(5mm)1.2 (A), SW2.2
- new net: JP7.2 (B), R23.1
- new net: JP14.2 (B), R14.1
- new net: JP15.2 (B), R15.1
- new net: C32.1, U4.6 (SS)
- new net CS_STM: R26.2
- new net DRDY_STM: U3.47 (~{DRDY})
- new net Din_STM: R28.2
- new net Dout_STM: U3.43 (DOUT)
- new net PWDN_STM: U3.35 (~{PWDN}), U3.36 (~{RESET})
- new net SCLK_STM: R25.2
- new net Strt_STM: R27.2
- new net Vout_5: C22.1, C23.1, C33.1, C34.1, C35.1, C36.1, R31.1, R31.2, R32.1, U3.19 (AVDD@1), U3.21 (AVDD@1), U3.22 (AVDD@1), U3.54 (AVDD1), U3.56 (AVDD@1), U3.59 (AVDD@2), U4.3 (VOUT), U4.4 (VOUT), U5.5 (VIN)
- no-connect marks 8 -> 20
Other:
- note added: "28 Feb 2026"
- note added: "ADS1299"
- note added: "Boost converter"
- note added: "Buck converter"
- note added: "Charging Unit"
- note added: "EEG Headband refined"
- note added: "Overcurrent and Overvoltage protection"
- note added: "USB-C receptacle"
- note added: "V1"
- moved on the sheet: C14, C15, C16, C7, D1, D2, J1, Q1, R2, R4, R5, R6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

Commit message: PCB ADS1299 and jumper connections
Parts:
- added J2, J3: Conn_01x10_Socket, Connector_PinSocket_2.54mm:PinSocket_1x10_P2.54mm_Vertical, symbol Connector:Conn_01x10_Socket
- renumbered U1 to U
Connections:
- net VDD is gone; now on net DGND: C1.1, C10.1, C11.1, C12.1, C13.1, C2.1, C3.1, C4.1, C5.1, C6.1, C8.1, C9.1, U.1 (VBAT), U.13 (VREF+), U.14 (VDDA), U.30 (VDD), U.33 (VDDRF), U.44 (VDDSMPS), U.45 (VDD), U.55 (VDDUSB), U.68 (VDD)
- net CS_STM: now also U.19 (PA4), J3.7 (Pin_7)
- net DGND: now also U.41 (VFBSMPS), U.43 (VLXSMPS), J2.5 (Pin_5), J2.6 (Pin_6), J3.2 (Pin_2), J3.3 (Pin_3)
- net DRDY_STM: now also U.16 (PA1), J3.5 (Pin_5)
- net Din_STM: now also U.22 (PA7), J3.10 (Pin_10)
- net Dout_STM: now also U.21 (PA6), J3.9 (Pin_9)
- net PWDN_STM: now also U.15 (PA0), J3.4 (Pin_4)
- net SCLK_STM: now also U.20 (PA5), J3.8 (Pin_8)
- net Strt_STM: now also U.23 (PA8), J3.6 (Pin_6)
- net Vout_5: now also J3.1 (Pin_1)
- net NRST: now reaches R1.1, SW1.1, U.8 (NRST)
- net NRST: now also J2.4 (Pin_4)
- net UART_TX: now reaches U.24 (PA9)
- net UART_TX: now also J2.7 (Pin_7)
- net UART_RX: now reaches U.51 (PA10)
- net UART_RX: now also J2.8 (Pin_8)
- net SWDIO: now reaches U.54 (PA13)
- net SWDIO: now also J2.2 (Pin_2)
- net SWCLK: now reaches U.56 (PA14)
- net SWCLK: now also J2.1 (Pin_1)
- net EXTRA1: now reaches U.6 (PB8)
- net EXTRA1: now also J2.10 (Pin_10)
- net SWO: now reaches U.63 (PB3)
- net SWO: now also J2.3 (Pin_3)
- net EXTRA2: now reaches U.7 (PB9)
- net EXTRA2: now also J2.9 (Pin_9)
Other:
- moved on the sheet: AE1, AE2, Bias, C1, C10, C11, C12, C13, C14, C15, C16, C17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
